File: Proyecto/PCB_files_kicad/project/power.sch (KiCad schematic (older format))
At the start: 21 parts, among them J7 Barrel_Jack, J8 USB_B_Micro, Q1 DMP3098LSS, U2 MCP73831-2-OT, U3 TPS61200DRC

Commit message: DONE: schematic v1.2
Parts:
- removed C4: 1uF, symbol Device:C
- removed R5: 2M, symbol Device:R_US
- removed R6: 140k 1%, symbol Device:R_US
- removed U2: MCP73831-2-OT, Package_TO_SOT_SMD:SOT-23-5, symbol Battery_Management:MCP73831-2-OT
- removed U3: TPS61200DRC, Package_SON:Texas_S-PVSON-N10_ThermalVias, symbol Regulator_Switching:TPS61200DRC
- added D5: CDBU0130L - 350mV, symbol Device:D_Schottky
- added R10: 15k, symbol Device:R_US
- added R11: 2k, symbol Device:R_US
- added U2: TP4056, symbol myLib:TP4056
- added U3: MT3608, Package_TO_SOT_SMD:SOT-23-6, symbol Regulator_Switching:MT3608
- C1, C2: value 4.7uF -> 10uF
- C3: value 4.7uF-X5R(check!) -> 22uF-X5R
- C5: value 22uF-X5R(check!) -> 22uF
- L1: value 2.2uH - LPS3015 -> 22uH; Mouser Link https://ar.mouser.com/ProductDetail/Coilcraft/LPS3015-222MR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 -> (none); Mouser Number 994-LPS3015-222MRC -> (none); Part Number LPS3015-222MRC -> (none)
- Q1: value DMP3098LSS -> IRF7240PBF; Mouser Link https://ar.mouser.com/ProductDetail/Infineon-Technologies/S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 -> (none); Mouser Number 726-SPD04P10PG -> ver en electrocomponentes!; Part Number SPD04P10P G -> (none)
- R3: value 2k -> 2.4k
Connections:
- net Earth: now also R3.1, R11.2, U2.1 (TEMP), U2.3 (GND), U3.2 (GND); no longer R3.2
- net OUTPUT_5V: now also D5.1 (K), R10.1
- net OUTPUT_BAT: now also U2.5 (BAT)
- net OUTPUT_MEASURE: now also U2.4 (VCC), U2.8 (CE)
- net at L1.2: now also D5.2 (A), U3.1 (SW)
- net at C3.1, L1.1, Q1.2 (D): now also U3.4 (EN), U3.5 (IN)
- new net: R3.2, U2.2 (PROG)
- new net: R10.2, R11.1, U3.3 (FB)
- no-connect marks 1 -> 2
Other:
- note added: "-4.5v > VGS"
- note added: "PullDown Resistor\n"
- note removed: "ANILIZAR SI EL CIRCUITO SE PODRIA HACER SIN BATERIA CON SUPER-CAP EN Vbat"
- note removed: "El divisor de tensión en el TPS6 está calculado para que la tensión de corte sea de 3.82V\n"
- note removed: "La resistencia en el MCP73831 está calculada para tener una corriente de carga de 500mA"
- note removed: "PullDown R"
- moved on the sheet: BT1, C1, C5, L1, R3
