File: Proyecto/PCB_files_kicad/project/project.sch (KiCad schematic (older format))
At the start: 16 parts, among them J1 Conn_01x08_Female, J2 S1, J3 S2, J4 Conn_01x08_Female, J5 Display, J6 HC06, U1 24AA64FT-I/OT

Commit message: DONE: schematic v1.2
Parts:
- added R5, R8: 2k, symbol Device:R_US
- added R6, R9: 3k, symbol Device:R_US
Connections:
- net BATT: now also R8.1
- net Earth: now also R6.2, R9.2
- net MEASURE: now also R5.1
- net blupill/SPI2_NSS: now also J4.1 (Pin_1)
- new net blupill/ADC12_IN0: R5.2, R6.1
- new net blupill/ADC12_IN1: R8.2, R9.1
- no-connect marks 3 -> 2
Other:
- note removed: "???"
